File: REF1662.kicad_pcb (KiCad board)
At the start: 2 copper layers, 53.6 x 67.1 mm, 26 parts, among them J1 USB_B_Mini, J2 SW_DPDT_x2, J3 System_Edge_Connector, J4 Game_Edge_Connector, SW1 SW_Push_Dual, U1 SST39VF800A, U2 EX256-TQ100, U3 NDS_Cart_Slot, U4 Cypress CY7C63743, Y1 40 MHz

Commit message: Add files via upload
Parts:
- U1: value SST39VF800A -> SST39VF400A/800A
Routing:
- net /VBUS: track 44.8 -> 45.4 mm
Other:
- board text added: "ACTEL eX256-F TQ100"
- board text removed: "Datel GBA/NDS 0602M3015"
Changed lines of the file:
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@@
         (effects (font (size 1 1) (thickness 0.15)))
     )
-    (fp_text value "SST39VF800A" (at -0.165 0.07 90) (layer "F.SilkS")
+    (fp_text value "SST39VF400A/800A" (at -0.165 0.07 90) (layer "F.SilkS")
         (effects (font (size 1 1) (thickness 0.15)))
     )
@@
     (effects (font (size 1 1) (thickness 0.15)))
   )
-  (gr_text "Datel\nGBA/NDS\n0602M3015" (at 160.357 107.002) (layer "F.SilkS")
+  (gr_text "ACTEL\neX256-F\nTQ100" (at 160.527 106.348) (layer "F.SilkS")
     (effects (font (size 1 1) (thickness 0.15)))
   )
@@
   (segment (start 151.1847 72.2563) (end 174.8975 72.2563) (width 0.15) (layer "B.Cu") (net 50))
   (segment (start 174.5254 75.945094) (end 174.5254 76.5556) (width 0.15) (layer "B.Cu") (net 50))
-  (segment (start 169.6764 84.4485) (end 169.6764 81.4806) (width 0.15) (layer "F.Cu") (net 51))
-  (segment (start 174.8908 72.2751) (end 151.9942 72.2751) (width 0.15) (layer "F.Cu") (net 51))
-  (segment (start 168.0929 86.032) (end 169.6764 84.4485) (width 0.15) (layer "F.Cu") (net 51))
+  (segment (start 151.9942 72.2751) (end 151.748 72.0289) (width 0.15) (layer "F.Cu") (net 51))
   (segment (start 170.442 80.715) (end 171.435 80.715) (width 0.15) (layer "F.Cu") (net 51))
-  (segment (start 167.066 86.032) (end 168.0929 86.032) (width 0.15) (layer "F.Cu") (net 51))
-  (segment (start 151.9942 72.2751) (end 151.748 72.0289) (width 0.15) (layer "F.Cu") (net 51))
-  (segment (start 175.6749 76.4751) (end 175.6749 73.0592) (width 0.15) (layer "F.Cu") (net 51))
+  (segment (start 168.195 86.032) (end 169.6764 84.5506) (width 0.15) (layer "F.Cu") (net 51))
   (segment (start 167.066 86.032) (end 165.7619 86.032) (width 0.15) (layer "F.Cu") (net 51))
   (segment (start 165.7619 86.032) (end 165.4319 85.702) (width 0.15) (layer "F.Cu") (net 51))
   (segment (start 164.53 85.702) (end 165.4319 85.702) (width 0.15) (layer "F.Cu") (net 51))
-  (segment (start 151.748 72.0289) (end 151.748 70.752) (width 0.15) (layer "F.Cu") (net 51))
-  (segment (start 171.435 80.715) (end 175.6749 76.4751) (width 0.15) (layer "F.Cu") (net 51))
+  (segment (start 167.066 86.032) (end 168.195 86.032) (width 0.15) (layer "F.Cu") (net 51))
   (segment (start 169.6764 81.4806) (end 170.442 80.715) (width 0.15) (layer "F.Cu") (net 51))
   (segment (start 175.6749 73.0592) (end 174.8908 72.2751) (width 0.15) (layer "F.Cu") (net 51))
-  (segment (start 167.066 85.402) (end 168.1179 85.402) (width 0.2) (layer "F.Cu") (net 52))
-  (segment (start 169.2019 81.2501) (end 168.655 81.2501) (width 0.2) (layer "F.Cu") (net 52))
-  (segment (start 152.7499 71.0039) (end 156.4231 71.0039) (width 0.2) (layer "F.Cu") (net 52))
-  (segment (start 168.655 82.177) (end 168.655 83.1039) (width 0.2) (layer "F.Cu") (net 52))
-  (segment (start 168.655 81.2501) (end 168.655 82.177) (width 0.2) (layer "F.Cu") (net 52))
-  (segment (start 168.1179 85.402) (end 168.1179 83.641) (width 0.2) (layer "F.Cu") (net 52))
-  (segment (start 171.5254 67.982) (end 174.5314 70.988) (width 0.2) (layer "F.Cu") (net 52))
-  (segment (start 159.445 67.982) (end 171.5254 67.982) (width 0.2) (layer "F.Cu") (net 52))
-  (segment (start 152.498 70.752) (end 152.7499 71.0039) (width 0.2) (layer "F.Cu") (net 52))
-  (segment (start 174.268733 76.183267) (end 169.2019 81.2501) (width 0.2) (layer "F.Cu") (net 52))
-  (segment (start 156.4231 71.0039) (end 159.445 67.982) (width 0.2) (layer "F.Cu") (net 52))
-  (segment (start 168.1179 83.641) (end 168.655 83.1039) (width 0.2) (layer "F.Cu") (net 52))
-  (segment (start 175.1004 76.183267) (end 174.268733 76.183267) (width 0.2) (layer "F.Cu") (net 52))
+  (segment (start 175.6749 76.4751) (end 175.6749 73.0592) (width 0.15) (layer "F.Cu") (net 51))
+  (segment (start 151.748 72.0289) (end 151.748 70.752) (width 0.15) (layer "F.Cu") (net 51))
+  (segment (start 174.8908 72.2751) (end 151.9942 72.2751) (width 0.15) (layer "F.Cu") (net 51))
+  (segment (start 171.435 80.715) (end 175.6749 76.4751) (width 0.15) (layer "F.Cu") (net 51))
+  (segment (start 169.6764 84.5506) (end 169.6764 81.4806) (width 0.15) (layer "F.Cu") (net 51))
+  (segment (start 168.051148 85.402) (end 168.655 84.798148) (width 0.4) (layer "F.Cu") (net 52))
+  (segment (start 172.213 68.031) (end 174.5314 70.3494) (width 0.4) (layer "F.Cu") (net 52))
+  (segment (start 156.424 71.157) (end 159.55 68.031) (width 0.4) (layer "F.Cu") (net 52))
+  (segment (start 152.903 71.157) (end 156.424 71.157) (width 0.4) (layer "F.Cu") (net 52))
+  (segment (start 167.066 85.402) (end 168.051148 85.402) (width 0.4) (layer "F.Cu") (net 52))
+  (segment (start 174.5314 70.3494) (end 174.5314 70.988) (width 0.4) (layer "F.Cu") (net 52))
+  (segment (start 173.716733 76.183267) (end 168.655 81.245) (width 0.4) (layer "F.Cu") (net 52))
+  (segment (start 152.498 70.752) (end 152.903 71.157) (width 0.4) (layer "F.Cu") (net 52))
+  (segment (start 168.655 84.798148) (end 168.655 82.177) (width 0.4) (layer "F.Cu") (net 52))
+  (segment (start 159.55 68.031) (end 172.213 68.031) (width 0.4) (layer "F.Cu") (net 52))
+  (segment (start 175.1004 76.183267) (end 173.716733 76.183267) (width 0.4) (layer "F.Cu") (net 52))
+  (segment (start 168.655 81.245) (end 168.655 82.177) (width 0.4) (layer "F.Cu") (net 52))
   (via (at 174.5314 70.988) (size 0.6) (drill 0.3) (layers "F.Cu" "B.Cu") (net 52))
   (via (at 175.1004 76.183267) (size 0.6) (drill 0.3) (layers "F.Cu" "B.Cu") (net 52))
-  (segment (start 175.1004 76.183267) (end 176.0156 75.268067) (width 0.2) (layer "B.Cu") (net 52))
-  (segment (start 176.0156 72.4722) (end 174.5314 70.988) (width 0.2) (layer "B.Cu") (net 52))
-  (segment (start 176.0156 75.268067) (end 176.0156 72.4722) (width 0.2) (layer "B.Cu") (net 52))
+  (segment (start 176.0801 72.5367) (end 174.5314 70.988) (width 0.4) (layer "B.Cu") (net 52))
+  (segment (start 175.1004 76.183267) (end 175.322733 76.183267) (width 0.4) (layer "B.Cu") (net 52))
+  (segment (start 176.0801 75.4259) (end 176.0801 72.5367) (width 0.4) (layer "B.Cu") (net 52))
+  (segment (start 175.322733 76.183267) (end 176.0801 75.4259) (width 0.4) (layer "B.Cu") (net 52))
   (segment (start 165.857 98.5234) (end 164.0689 96.7353) (width 0.15) (layer "F.Cu") (net 53))
   (segment (start 165.857 99.3395) (end 165.857 98.5234) (width 0.15) (layer "F.Cu") (net 53))
