File: REF1662.kicad_sch (KiCad schematic)
At the start: 25 parts, among them J1 USB_B_Mini, J2 SW_DPDT_x2, J3 System_Edge_Connector, J4 Game_Edge_Connector, SW1 SW_Push_Dual, U1 SST39VF800A-70-4C-EKE, U2 EX256-TQ100, U3 NDS_Cart_Slot, U4 Cypress CY7C63743, Y1 40 MHz

Commit message: Add files via upload
Parts:
- U1: value SST39VF800A-70-4C-EKE -> SST39VF400A-70-4C-EKE
Changed lines of the file:
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@@
   (symbol (lib_id "GBA:SST39VF200A-70-4C-EKE") (at 38.1 26.67 0) (unit 1)
     (in_bom yes) (on_board yes) (dnp no) (fields_autoplaced)
-    (property "Reference" "U1" (at 53.34 19.05 0)
+    (property "Reference" "U1" (at 53.34 20.32 0)
       (effects (font (size 1.27 1.27)))
     )
-    (property "Value" "SST39VF800A-70-4C-EKE" (at 53.34 21.59 0)
+    (property "Value" "SST39VF400A-70-4C-EKE" (at 53.34 22.86 0)
       (effects (font (size 1.27 1.27)))
     )
